File: Encoder.kicad_sch (KiCad schematic)
At the start: 17 parts, among them J1 Conn_01x05_Pin, SW1 RotaryEncoder_Switch_MP, U1 74LVC3G14

Commit message: Layout done
Parts:
- C1, C2, C3, C4, J1, R1, R2, R3, R4, R5, R6: now left out of the parts list
- SW1: LCSC (none) -> C470596
- U1: footprint Package_SO:SSOP-8_3.9x5.05mm_P1.27mm -> Package_SO:VSSOP-8_2.3x2mm_P0.5mm; LCSC (none) -> C98856
Connections:
- net BTN: now also SW1.S2; no longer SW1.S1
- net GND: now also SW1.S1; no longer SW1.S2
Changed lines of the file:
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@@
-	(wire
-		(pts
-			(xy 137.16 91.44) (xy 137.16 97.79)
-		)
-		(stroke
-			(width 0)
-			(type default)
-		)
-	)
 	(wire
 		(pts
@@
 	(wire
 		(pts
-			(xy 135.89 91.44) (xy 137.16 91.44)
+			(xy 135.89 91.44) (xy 139.7 91.44)
 		)
 		(stroke
@@
 	(wire
 		(pts
+			(xy 142.24 97.79) (xy 142.24 86.36)
+		)
+		(stroke
+			(width 0)
+			(type default)
+		)
+	)
+	(wire
+		(pts
 			(xy 36.83 99.06) (xy 36.83 101.6)
 		)
@@
 	(wire
 		(pts
-			(xy 137.16 97.79) (xy 128.27 97.79)
+			(xy 128.27 97.79) (xy 142.24 97.79)
 		)
 		(stroke
@@
 		)
 	)
-	(label "BTN"
-		(at 142.24 86.36 180)
-		(effects
-			(font
-				(size 1.27 1.27)
-			)
-			(justify right bottom)
-		)
-	)
 	(label "Debounced.A"
 		(at 31.75 91.44 0)
@@
 		)
 	)
+	(label "BTN"
+		(at 139.7 91.44 180)
+		(effects
+			(font
+				(size 1.27 1.27)
+			)
+			(justify right bottom)
+		)
+	)
 	(label "A"
 		(at 175.26 95.25 0)
@@
 		(unit 1)
 		(exclude_from_sim no)
-		(in_bom yes)
+		(in_bom no)
 		(on_board yes)
 		(dnp no)
@@
 		(unit 1)
 		(exclude_from_sim no)
-		(in_bom yes)
+		(in_bom no)
 		(on_board yes)
 		(dnp no)
@@
 			)
 		)
-		(property "Footprint" "Package_SO:SSOP-8_3.9x5.05mm_P1.27mm"
+		(property "Footprint" "Package_SO:VSSOP-8_2.3x2mm_P0.5mm"
 			(at 203.2 95.25 0)
 			(effects
@@
 			)
 		)
+		(property "LCSC" "C98856"
+			(at 204.47 95.25 0)
+			(effects
+				(font
+					(size 1.27 1.27)
+				)
+				(hide yes)
+			)
+		)
 		(pin "1"
 		)
@@
 		(unit 1)
 		(exclude_from_sim no)
-		(in_bom yes)
+		(in_bom no)
 		(on_board yes)
 		(dnp no)
@@
 			)
 		)
+		(property "LCSC" "C470596"
+			(at 128.27 88.9 0)
+			(effects
+				(font
+					(size 1.27 1.27)
+				)
+				(hide yes)
+			)
+		)
 		(pin "S1"
 		)
@@
 			)
 		)
-		(property "Footprint" "Package_SO:SSOP-8_3.9x5.05mm_P1.27mm"
+		(property "Footprint" "Package_SO:VSSOP-8_2.3x2mm_P0.5mm"
 			(at 203.2 120.65 0)
 			(effects
@@
 		)
 		(property "Description" "Triple NOT Gate Schmitt, Low-Voltage CMOS"
+			(at 204.47 120.65 0)
+			(effects
+				(font
+					(size 1.27 1.27)
+				)
+				(hide yes)
+			)
+		)
+		(property "LCSC" "C98856"
 			(at 204.47 120.65 0)
 			(effects
@@
 			)
 		)
-		(property "Footprint" "Package_SO:SSOP-8_3.9x5.05mm_P1.27mm"
+		(property "Footprint" "Package_SO:VSSOP-8_2.3x2mm_P0.5mm"
 			(at 81.28 40.64 0)
 			(effects
@@
 			)
 		)
+		(property "LCSC" "C98856"
+			(at 82.55 40.64 0)
+			(effects
+				(font
+					(size 1.27 1.27)
+				)
+				(hide yes)
+			)
+		)
 		(pin "1"
 		)
@@
 		(unit 1)
 		(exclude_from_sim no)
-		(in_bom yes)
+		(in_bom no)
 		(on_board yes)
 		(dnp no)
@@
 		(unit 1)
 		(exclude_from_sim no)
-		(in_bom yes)
+		(in_bom no)
 		(on_board yes)
 		(dnp no)
@@
 		(unit 1)
 		(exclude_from_sim no)
-		(in_bom yes)
+		(in_bom no)
 		(on_board yes)
 		(dnp no)
@@
 		(unit 1)
 		(exclude_from_sim no)
-		(in_bom yes)
+		(in_bom no)
 		(on_board yes)
 		(dnp no)
@@
 			)
 		)
-		(property "Footprint" "Package_SO:SSOP-8_3.9x5.05mm_P1.27mm"
+		(property "Footprint" "Package_SO:VSSOP-8_2.3x2mm_P0.5mm"
 			(at 201.93 69.85 0)
 			(effects
@@
 		)
 		(property "Description" "Triple NOT Gate Schmitt, Low-Voltage CMOS"
+			(at 203.2 69.85 0)
+			(effects
+				(font
+					(size 1.27 1.27)
+				)
+				(hide yes)
+			)
+		)
+		(property "LCSC" "C98856"
 			(at 203.2 69.85 0)
 			(effects
@@
 		(unit 1)
 		(exclude_from_sim no)
-		(in_bom yes)
+		(in_bom no)
 		(on_board yes)
 		(dnp no)
@@
 		(unit 1)
 		(exclude_from_sim no)
-		(in_bom yes)
+		(in_bom no)
 		(on_board yes)
 		(dnp no)
@@
 		(unit 1)
 		(exclude_from_sim no)
-		(in_bom yes)
+		(in_bom no)
 		(on_board yes)
 		(dnp no)
@@
 		(unit 1)
 		(exclude_from_sim no)
-		(in_bom yes)
-		(on_board yes)
-		(dnp no)
+		(in_bom no)
+		(on_board yes)
+		(dnp no)
